File: lego_motors_booster_1x4-.sch (EAGLE design)
At the start: 21 parts, among them Q1 IRF4905, Q3 BS170T, Q5 BUZ11BV, X1 NXT-SOCKET, X2 NXT-SOCKET, X3 NXT-SOCKET, X4 NXT-SOCKET, X5 NXT-SOCKET

Commit message: mirrored + maybe some minor improvements
Connections:
- removed net N$11: X4.4
- removed net N$12: X4.5
- removed net N$13: X4.6
- removed net N$17: X5.4
- removed net N$18: X5.5
- removed net N$19: X5.6
- removed net N$5: X3.4
- removed net N$6: X3.5
- removed net N$7: X3.6
- net GND: no longer X3.3, X4.3, X5.3
Changed lines of the file:
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@@
 <?xml version="1.0" encoding="utf-8"?>
 <!DOCTYPE eagle SYSTEM "eagle.dtd">
-<eagle version="7.7.0">
+<eagle version="7.2.0">
 <drawing>
 <settings>
@@
 </segment>
 <segment>
-<wire x1="106.68" y1="20.32" x2="93.98" y2="20.32" width="0.1524" layer="91"/>
-<label x="93.98" y="20.32" size="1.778" layer="95"/>
-<pinref part="X3" gate="G$1" pin="3"/>
-</segment>
-<segment>
-<wire x1="106.68" y1="-15.24" x2="93.98" y2="-15.24" width="0.1524" layer="91"/>
-<label x="93.98" y="-15.24" size="1.778" layer="95"/>
-<pinref part="X4" gate="G$1" pin="3"/>
-</segment>
-<segment>
-<wire x1="106.68" y1="-48.26" x2="93.98" y2="-48.26" width="0.1524" layer="91"/>
-<label x="93.98" y="-48.26" size="1.778" layer="95"/>
-<pinref part="X5" gate="G$1" pin="3"/>
-</segment>
-<segment>
 <wire x1="30.48" y1="83.82" x2="30.48" y2="73.66" width="0.1524" layer="91"/>
 <label x="30.48" y="76.2" size="1.778" layer="95" rot="R90"/>
@@
 </segment>
 </net>
-<net name="N$5" class="0">
-<segment>
-<wire x1="106.68" y1="17.78" x2="93.98" y2="17.78" width="0.1524" layer="91"/>
-<label x="93.98" y="17.78" size="1.778" layer="95"/>
-<pinref part="X3" gate="G$1" pin="4"/>
-</segment>
-</net>
-<net name="N$6" class="0">
-<segment>
-<wire x1="106.68" y1="15.24" x2="93.98" y2="15.24" width="0.1524" layer="91"/>
-<label x="93.98" y="15.24" size="1.778" layer="95"/>
-<pinref part="X3" gate="G$1" pin="5"/>
-</segment>
-</net>
-<net name="N$7" class="0">
-<segment>
-<wire x1="106.68" y1="12.7" x2="93.98" y2="12.7" width="0.1524" layer="91"/>
-<label x="93.98" y="12.7" size="1.778" layer="95"/>
-<pinref part="X3" gate="G$1" pin="6"/>
-</segment>
-</net>
-<net name="N$11" class="0">
-<segment>
-<wire x1="106.68" y1="-17.78" x2="93.98" y2="-17.78" width="0.1524" layer="91"/>
-<label x="93.98" y="-17.78" size="1.778" layer="95"/>
-<pinref part="X4" gate="G$1" pin="4"/>
-</segment>
-</net>
-<net name="N$12" class="0">
-<segment>
-<wire x1="106.68" y1="-20.32" x2="93.98" y2="-20.32" width="0.1524" layer="91"/>
-<label x="93.98" y="-20.32" size="1.778" layer="95"/>
-<pinref part="X4" gate="G$1" pin="5"/>
-</segment>
-</net>
-<net name="N$13" class="0">
-<segment>
-<wire x1="106.68" y1="-22.86" x2="93.98" y2="-22.86" width="0.1524" layer="91"/>
-<label x="93.98" y="-22.86" size="1.778" layer="95"/>
-<pinref part="X4" gate="G$1" pin="6"/>
-</segment>
-</net>
-<net name="N$17" class="0">
-<segment>
-<wire x1="106.68" y1="-50.8" x2="93.98" y2="-50.8" width="0.1524" layer="91"/>
-<label x="93.98" y="-50.8" size="1.778" layer="95"/>
-<pinref part="X5" gate="G$1" pin="4"/>
-</segment>
-</net>
-<net name="N$18" class="0">
-<segment>
-<wire x1="106.68" y1="-53.34" x2="93.98" y2="-53.34" width="0.1524" layer="91"/>
-<label x="93.98" y="-53.34" size="1.778" layer="95"/>
-<pinref part="X5" gate="G$1" pin="5"/>
-</segment>
-</net>
-<net name="N$19" class="0">
-<segment>
-<wire x1="106.68" y1="-55.88" x2="93.98" y2="-55.88" width="0.1524" layer="91"/>
-<label x="93.98" y="-55.88" size="1.778" layer="95"/>
-<pinref part="X5" gate="G$1" pin="6"/>
-</segment>
-</net>
